File: POE_hat_and_USB.kicad_pcb (KiCad board)
At the start: 2 copper layers, 100 x 30 mm, 58 parts, among them J1 GPIO_CONNECTOR, J2 RJHSE-5385, J3 PIR Motion Sensor, J4 DH22T, J8 USB_B_Micro, Q1 DMG1012UW-7, U2 RTL8152B-VB, Y2 25 MHz 30ppm (HELE(Harmony El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

Commit message: v1.1.0 prerelease.
Parts:
- added ?: , user-footprints:LOGO_eLAB, F.Cu at (110.9, 96.3)
Routing:
- net /VDD10: track 34.9 -> 34.6 mm, vias 4 -> 3
- net GND: vias 29 -> 93
